File: hardware/LFX_FC_R1/LFX_FC_R1.kicad_pcb (KiCad board)
At the start: 4 copper layers, 46 x 46 mm, 84 parts, among them J1 SM08B-SRSS-TB, J10 M4 pad, J11 M1 GND, J12 M2 GND, J13 M3 GND, J14 M4 GND, J2 VBAT pad, J3 GND pad, J4 SM03B-SRSS-TB, J5 SM04B-SRSS-TB, J6 SM02B-SRSS-TB, J7 M1 pad, J8 M2 pad, J9 M3 pad, Q1 AO3400A, U1 TPS54360DDA, U2 LM66100DCK, U3 TLV75533PDBV, U4 ICM-42688-P, U5 BMP390, U6 TPD4E05U06DQA, U7 TPD4E05U06DQA

Commit message: hardware: RC receiver port (ELRS/CRSF) on UART2 instead of debug console
- J4 becomes a 4-pin JST-SH RC port: 1 5V, 2 GND, 3 TX (to receiver RX),
  4 RX (from receiver TX, CRSF 420000 baud), same order as the GPS port
- R24 1k pull-up on RC_RX to the module's 3V3 (pin 3): ESP-based ELRS
  receivers stall in the bootloader if that line is low at power-up
  (expresslrs.org receiver wiring guide)
- TP5/TP6 on RC_TX/RC_RX: console tap with the receiver unplugged
- UART2 has its own fractional divider (clk-rv1106.c:441), 420000 x 16 =
  24 MHz x 7/25; not yet measured
- docs: RC path goes through Linux, MCU failsafe on heartbeat loss; the
  console has to leave UART2 in software (fiq-debugger, earlycon)
- ERC 0, DRC 0 / 0 unconnected / 0 parity errors

Co-Authored-By: Claude Opus 5.5 <noreply@anthropic.com>
Parts:
- added R24: 1k, Resistor_SMD:R_0402_1005Metric, F.Cu at (11.2, 9.40)
- added TP5: TP, LFX:TestPad_1.0mm, F.Cu at (6.40, 28.4)
- added TP6: TP, LFX:TestPad_1.0mm, F.Cu at (9.20, 28.4)
- J4: value SM03B-SRSS-TB -> SM04B-SRSS-TB; footprint Connector_JST:JST_SH_SM03B-SRSS-TB_1x03-1MP_P1.00mm_Horizontal -> Connector_JST:JST_SH_SM04B-SRSS-TB_1x04-1MP_P1.00mm_Horizontal
Connections:
- net DBG_RX renamed RC_RX
- net DBG_TX renamed RC_TX
- J4 pad 1: DBG_TX_X -> +5V
- J4 pad 2: DBG_RX_X -> GND
- J4 pad 3: GND -> RC_TX_X
- MOD1 pad 3: unconnected-(MOD1-3V3_O-Pad3) -> 3V3_MOD
- R8 pad 2: DBG_TX_X -> RC_TX_X
- R9 pad 1: DBG_RX_X -> RC_RX_X
- U7 pad 1: DBG_TX_X -> RC_TX_X
- U7 pad 2: DBG_RX_X -> RC_RX_X
Routing:
- net +5V: track 122.6 -> 163.8 mm, vias 7 -> 6
- net ESC_M2: track 62.8 -> 89.5 mm
- net ESC_M1: track 50.9 -> 71.1 mm
- net RC_TX: track 15.2 -> 33.7 mm, vias 0 -> 1
- net DBG_TX_X: track 17.1 -> 0.00 mm
- net DBG_RX_X: track 15.1 -> 0.00 mm
- net RC_RX_X: track 0.00 -> 15.0 mm, vias 0 -> 3
- net ESC_M3: track 71.1 -> 56.6 mm, vias 1 -> 2
- net RC_RX: track 11.0 -> 24.6 mm, vias 0 -> 1
- net RC_TX_X: track 0.00 -> 13.4 mm, vias 0 -> 2
- net 3V3_MOD: track 0.00 -> 3.89 mm
- net ESC_M4: track 38.4 -> 35.2 mm, vias 2 -> 3
- net ADC_VBAT: track 42.6 -> 45.6 mm, vias 0 -> 1
- net GPS_RX_X: track 8.04 -> 9.80 mm
Other:
- board text added: "RC"
- board text removed: "DBG"

Commit message: hardware: LFX_LTE_R1 stacked LTE + GNSS board, FC link on J5
New 46 x 46 mm board hardware/LFX_LTE_R1 (same 39 mm M3 pattern, stacks on
the flight controller, all parts on the top side):
- Lierda NT26-KCN E LTE Cat.1 bis + GNSS (order the GPS + BDS variant);
  symbol and LCC/LGA-109 land pattern drawn from the Lierda hardware design
  manual Rev1.0 (table 2-5, fig. 2-2, fig. 8-3)
- TLV62569 buck +5V -> 3.8 V (modem VBAT 3.3-4.5 V), In2 +3V8 plane,
  2 x 47 uF + 100n / 33p / 8p2 at VBAT; TLV75533 3.3 V for the translators
- UART 3.3 <-> 1.8 V by 2 x SN74LVC1T45 (Hi-Z while the modem is off)
- Luckfox reflashes the modem: RESET_N via AO3400A, USB_BOOT via 1k from the
  1.8 V BOOT pin; USB / debug test pads for a PC rescue
- hinged nano-SIM with 22R / 33p / TPD4E05U06, LTE and GNSS U.FL with pi
  match, 50 ohm 0.35 mm feeds, active GNSS antenna bias
- ERC 0, DRC 0 violations / 0 unconnected / 0 parity

LFX_FC_R1 stays 46 x 46 mm:
- J5 GPS (JST-SH 4) -> LTE board link (JST-SH 10): 5V x2, GND x2, UART3,
  RESET (pin 18), BOOT (pin 20), buzzer gate, ESC current
- buzzer gate and ESC current now come from the modem's GPIO1 / ADC0
- ERC 0, DRC 0 violations / 0 unconnected / 0 parity

Shared: NT26-KCN and SIM_Card_Shield in the LFX library, stacked symbol
pins in gen_sch, route_pcb creates pcb/.  README and architecture docs
updated.

Co-Authored-By: Claude Opus 5.5 <noreply@anthropic.com>
Parts:
- removed C22: 100n/16V, Capacitor_SMD:C_0402_1005Metric
- removed D6: BAT54S, Package_TO_SOT_SMD:SOT-23
- J5: value SM04B-SRSS-TB -> SM10B-SRSS-TB; footprint Connector_JST:JST_SH_SM04B-SRSS-TB_1x04-1MP_P1.00mm_Horizontal -> Connector_JST:JST_SH_SM10B-SRSS-TB_1x10-1MP_P1.00mm_Horizontal
- R18: value 10k 1% -> 33R; footprint Resistor_SMD:R_0603_1608Metric -> Resistor_SMD:R_0402_1005Metric
- R19: value 12k 1% -> 33R; footprint Resistor_SMD:R_0603_1608Metric -> Resistor_SMD:R_0402_1005Metric
- moved R18 12.3 mm to (34.4, 11.6), turned to 90 degrees
- moved R19 11.2 mm to (34.4, 6.47), turned to 90 degrees
- moved U6 3.30 mm to (37.4, 29.6)
- moved J5 2.40 mm to (42.5, 30.3)
Connections:
- net GPS_RX renamed LTE_RX
- net GPS_TX renamed LTE_TX
- J5 pad 2: GND -> +5V
- J5 pad 3: GPS_TX_X -> GND
- J5 pad 4: GPS_RX_X -> GND
- MOD1 pad 18: BUZ_CTRL -> LTE_RST
- MOD1 pad 20: ADC_CUR -> LTE_BOOT
- R18 pad 1: ESC_CUR -> LTE_RST
- R18 pad 2: ADC_CUR -> LTE_RST_X
- R19 pad 1: ADC_CUR -> LTE_BOOT
- R19 pad 2: GND -> LTE_BOOT_X
- R20 pad 2: GPS_TX_X -> LTE_TX_X
- R21 pad 1: GPS_RX_X -> LTE_RX_X
- U6 pad 1: GPS_TX_X -> LTE_TX_X
- U6 pad 2: GPS_RX_X -> LTE_RX_X
Routing:
- net VSYS: track 6.90 -> 98.0 mm, vias 9 -> 17
- net ESC_M2: track 89.5 -> 55.8 mm, vias 1 -> 3
- net LTE_BOOT_X: track 0.00 -> 24.9 mm, vias 0 -> 1
- net LTE_RST_X: track 0.00 -> 23.1 mm, vias 0 -> 1
- net ADC_CUR: track 19.8 -> 0.00 mm
- net LTE_RX_X: track 0.00 -> 15.9 mm, vias 0 -> 2
- net ESC_M1: track 71.1 -> 56.4 mm, vias 3 -> 1
- net ESC_CUR: track 44.3 -> 29.8 mm, vias 2 -> 1
- net GPS_RX_X: track 9.80 -> 0.00 mm
- net BUZ_CTRL: track 14.2 -> 5.73 mm
- net LTE_TX_X: track 0.00 -> 7.82 mm
- net RC_TX_X: track 13.4 -> 21.2 mm
- net SPI_MISO: track 26.4 -> 19.0 mm, vias 1 -> 2
- net RC_TX: track 33.7 -> 26.3 mm, vias 1 -> 2
- net ESC_M3: track 56.6 -> 49.7 mm
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Other:
- board text added: "B"
- board text added: "C"
- board text added: "LTE"
- board text added: "Z"
- board text removed: "GPS"
