File: hardware/LFX_FC_R1/sch/02_power.kicad_sch (KiCad schematic)
At the start: 35 parts, among them J2 VBAT pad, J3 GND pad, U1 TPS54360DDA, U2 LM66100DCK, U3 TLV75533PDBV

Commit message: hardware: LFX_FC_R1 46x46 layout routed, DRC + parity clean
- 46 x 46 mm, M3 NPTH holes in the corners (39 x 39 mm pattern),
  JST-SH connectors on the edges, ESC S/G solder pads at the four corners
- IMU turned 90 deg so CS/SCK/MOSI/MISO face module pins 6..9 in order;
  the four lines are drawn (route_critical.hand_route_imu), not searched
- via/track keep-outs under the IMU and barometer bodies, 0.5 mm routing
  keep-out round the board rim
- EN divider re-laid as one column (U1.3 -> R1 -> R2 -> D2)
- VBAT divider top resistor moved to the battery end; only the divided
  node crosses the board
- GPS ESD at J5, series resistors at the module pins, no crossings
- router: hole-to-hole on same-net vias, 5 um freerouting clearance margin,
  off-plane fan-out vias removed
- schematic parity: global labels, library nicknames, MountingPin
  connectors, #FLG power flags, BOM exclusion for bare pads
- ERC 0, DRC 0 violations / 0 unconnected / 0 footprint errors
  (--schematic-parity)

Co-Authored-By: Claude Opus 5.5 <noreply@anthropic.com>
Parts:
- removed C3: 10u/50V, Capacitor_SMD:C_1210_3225Metric, symbol Device:C
- C1, C2: value 2u2/100V -> 2u2/100V X7S; footprint Capacitor_SMD:C_1210_3225Metric -> Capacitor_SMD:C_1206_3216Metric
- D1: value SM6T33A -> SMAJ33A; footprint Diode_SMD:D_SMB -> Diode_SMD:D_SMA; symbol Diode:SM6T33A -> Diode:SMAJ33A
- D3: value B560C -> B360B; footprint Diode_SMD:D_SMC -> Diode_SMD:D_SMB
- J2, J3, TP1, TP2, TP3: now left out of the parts list
- L1: footprint Inductor_SMD:L_Coilcraft_XAL6060-XXX -> Inductor_SMD:L_Coilcraft_XAL5050-XXX
Connections:
- net VBAT: now also D1.1 (A1)
- net VBAT_F: no longer D1.1 (A1)
Other:
- moved on the sheet: C1, C4, D1, FB1
