File: hardware/LFX_FC_R2/LFX_FC_R2.kicad_pcb (KiCad board)
At the start: 4 copper layers, 50 x 50 mm, 139 parts, among them J10 M4 pad, J11 M1 GND, J12 M2 GND, J13 M3 GND, J14 M4 GND, J15 SIM8060-6-0-14-00, J16 U.FL-R-SMT-1, J17 U.FL-R-SMT-1, J2 VBAT pad, J3 GND pad, J4 SM04B-SRSS-TB, J6 SM02B-SRSS-TB, J7 M1 pad, J8 M2 pad, J9 M3 pad, Q1 AO3400A, Q2 AO3400A, Q3 MMBT3904, U1 TPS54360DDA, U10 SN74LVC1T45DBV, U11 TLV62569DBV, U12 TPD4E05U06DQA, U2 LM66100DCK, U3 TLV75533PDBV, U4 ICM-42688-P, U5 BMP390, U7 TPD4E05U06DQA, U8 NT26-KCN E (GPS+BDS), U9 SN74LVC1T45DBV

Commit message: hardware: LFX_FC_R2 GPS port J18 (ATGM336H / NEO-M8N class) on UART5
- J18: JST-SH 4-pin at the left edge, 1 +5V, 2 GND, 3 NC, 4 module TXD ->
  board RX.  MOD1 pin 14 (GPIO1_D2) becomes UART5_RX_M1, 33R + TPD1E05U06 ESD.
- Baro chip select moves to pin 15 (GPIO1_D3, MCU GPIO); IMU INT1 dropped
  (polled).
- +5V to J18 hand-routed from J4 on B.Cu along the board edge (x 0.75), so it
  walls nothing in.
- Hand routes for the connections the router kept leaving open: SIM RST/CLK
  (U12 channels swapped so they no longer cross), BUZ_CTRL, the U2 +5V
  escape, LTE_1V8 between U9/U10 (paths taken from dc53508).
- gen_sch keeps the board rules in kicad_pro; clean_stubs removes dangling
  vias; Freerouting runs as a background UI element on macOS.
- DRC: 0 violations, 0 unconnected, schematic parity clean; ERC 0.

Co-Authored-By: Claude Opus 5.5 <noreply@anthropic.com>
Parts:
- added J18: SM04B-SRSS-TB, Connector_JST:JST_SH_SM04B-SRSS-TB_1x04-1MP_P1.00mm_Horizontal, F.Cu at (3.55, 36.9)
- added R44: 33R, Resistor_SMD:R_0402_1005Metric, B.Cu at (9.80, 37.2)
- added U13: TPD1E05U06DPY, Package_SON:Texas_DPY0002A_0.6x1mm_P0.65mm, F.Cu at (8.20, 37.2)
- moved TP13 7.25 mm to (8.65, 32.1)
- moved C37 7.25 mm to (11.3, 31.8)
- moved C38 4.92 mm to (11.3, 33.8)
- moved R27 4.25 mm to (9.98, 35.0)
- moved R11 4.18 mm to (28.4, 17.0)
- moved C45 4.10 mm to (13.4, 33.5)
- moved L3 1.65 mm to (7.15, 39.6)
Connections:
- MOD1 pad 14: BARO_CS -> GPS_RX
- MOD1 pad 15: IMU_INT1 -> BARO_CS
- U12 pad 4: SIM_CLK -> SIM_RST
- U12 pad 5: SIM_RST -> SIM_CLK
- U4 pad 4: IMU_INT1 -> unconnected-(U4-INT1-Pad4)
Routing:
- net +3V3S: track 74.5 -> 28.1 mm, vias 18 -> 13
- net EN5: track 70.6 -> 24.7 mm, vias 0 -> 2
- net LTE_TX: track 70.2 -> 29.5 mm
- net GPS_RX: track 0.00 -> 31.0 mm
- net +5V: track 179.8 -> 207.6 mm
- net LTE_1V8: track 102.4 -> 78.0 mm, vias 4 -> 6
- net GNSS_VCC: track 9.73 -> 30.1 mm, vias 0 -> 4
- net LTE_USB_DM: track 48.5 -> 29.4 mm
- net LTE_RX: track 44.1 -> 60.1 mm
- net LTE_USB_VBUS: track 39.4 -> 25.1 mm
- net SIM_VDD: track 41.1 -> 29.1 mm, vias 1 -> 4
- net LTE_PWRKEY: track 22.1 -> 10.7 mm
- net LTE_BOOT_M: track 37.9 -> 48.2 mm
- net IMU_INT1: track 9.68 -> 0.00 mm
- net BUZ_N: track 20.8 -> 12.4 mm
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Other:
- board text added: "GPS"

Commit message: hardware: LFX_FC_R2 J18 as a 5-pin 2.54 mm header for the ATGM336H module
The JST-SH 4 GPS port becomes a right-angle 1x05 header at the left edge,
pin for pin with the 5-pin ATGM336H module (VCC GND TXD RXD PPS), so a
straight Dupont lead plugs in. Module TXD goes to UART5_RX as before;
RXD and PPS stay open (no Luckfox pins left).

New LFX footprint PinHeader_1x05_P2.54mm_EdgeHorizontal (stock 3D model
turned 180 degrees). Probe pads TP8/TP9 move to the bottom beside it.
Board edited in place from the routed R2: DRC 0 / unconnected 0 /
parity 0, ERC 0. 3D renders refreshed.

Co-Authored-By: Claude Opus 5.5 <noreply@anthropic.com>
Parts:
- J18: value SM04B-SRSS-TB -> PinHeader 1x05 2.54 RA; footprint Connector_JST:JST_SH_SM04B-SRSS-TB_1x04-1MP_P1.00mm_Horizontal -> LFX:PinHeader_1x05_P2.54mm_EdgeHorizontal
- TP8, TP9: moved to B.Cu
- moved J18 7.94 mm to (4.30, 29.0), turned to 0 degrees
- moved TP9 5.15 mm to (1.40, 34.1), turned to 180 degrees
- moved TP8 2.00 mm to (1.40, 31.6), turned to 180 degrees
Connections:
- J18 pad 3: unconnected-(J18-Pin_3-Pad3) -> GPS_RX_X
- J18 pad 4: GPS_RX_X -> unconnected-(J18-Pin_4-Pad4)
Routing:
- net +5V: track 207.6 -> 202.9 mm, vias 14 -> 13
- net LTE_USB_DP: track 32.7 -> 36.6 mm, vias 3 -> 2
- net GPS_RX_X: track 4.67 -> 7.00 mm
- net LTE_1V8: track 78.0 -> 79.2 mm, vias 6 -> 7
- net GND: track 49.0 -> 48.5 mm, vias 125 -> 122
Other:
- board text added: "P"
