File: hardware/LFX_FC_R2/sch/04_sensors.kicad_sch (KiCad schematic)
At the start: 9 parts, among them U4 ICM-42688-P, U5 BMP390

Commit message: hardware: LFX_FC_R2 GPS port J18 (ATGM336H / NEO-M8N class) on UART5
- J18: JST-SH 4-pin at the left edge, 1 +5V, 2 GND, 3 NC, 4 module TXD ->
  board RX.  MOD1 pin 14 (GPIO1_D2) becomes UART5_RX_M1, 33R + TPD1E05U06 ESD.
- Baro chip select moves to pin 15 (GPIO1_D3, MCU GPIO); IMU INT1 dropped
  (polled).
- +5V to J18 hand-routed from J4 on B.Cu along the board edge (x 0.75), so it
  walls nothing in.
- Hand routes for the connections the router kept leaving open: SIM RST/CLK
  (U12 channels swapped so they no longer cross), BUZ_CTRL, the U2 +5V
  escape, LTE_1V8 between U9/U10 (paths taken from dc53508).
- gen_sch keeps the board rules in kicad_pro; clean_stubs removes dangling
  vias; Freerouting runs as a background UI element on macOS.
- DRC: 0 violations, 0 unconnected, schematic parity clean; ERC 0.

Co-Authored-By: Claude Opus 5.5 <noreply@anthropic.com>
Connections:
- net IMU_INT1: no longer names the net of U4.4 (INT1)
- no-connect marks 1 -> 2
