File: hardware/LFX_FC_R2/sch/07_lte_rf.kicad_sch (KiCad schematic)
At the start: 23 parts, among them J15 SIM8060-6-0-14-00, J16 U.FL-R-SMT-1, J17 U.FL-R-SMT-1, U12 TPD4E05U06DQA

Commit message: hardware: LFX_FC_R2 GPS port J18 (ATGM336H / NEO-M8N class) on UART5
- J18: JST-SH 4-pin at the left edge, 1 +5V, 2 GND, 3 NC, 4 module TXD ->
  board RX.  MOD1 pin 14 (GPIO1_D2) becomes UART5_RX_M1, 33R + TPD1E05U06 ESD.
- Baro chip select moves to pin 15 (GPIO1_D3, MCU GPIO); IMU INT1 dropped
  (polled).
- +5V to J18 hand-routed from J4 on B.Cu along the board edge (x 0.75), so it
  walls nothing in.
- Hand routes for the connections the router kept leaving open: SIM RST/CLK
  (U12 channels swapped so they no longer cross), BUZ_CTRL, the U2 +5V
  escape, LTE_1V8 between U9/U10 (paths taken from dc53508).
- gen_sch keeps the board rules in kicad_pro; clean_stubs removes dangling
  vias; Freerouting runs as a background UI element on macOS.
- DRC: 0 violations, 0 unconnected, schematic parity clean; ERC 0.

Co-Authored-By: Claude Opus 5.5 <noreply@anthropic.com>
Connections:
- net SIM_CLK: now also U12.5 (D2-); no longer U12.4 (D2+)
- net SIM_RST: now also U12.4 (D2+); no longer U12.5 (D2-)
Changed lines of the file:
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@@
 		(unit 1)
 		(exclude_from_sim no) (in_bom no) (on_board yes) (dnp no)
-		(property "Reference" "#PWR0140"
+		(property "Reference" "#PWR0144"
 			(at 60.96 34.29 0)
 			(effects (font (size 1.27 1.27)) (hide yes))
@@
 			(project "LFX_FC_R2"
 				(path "/9564b83f-500d-c692-1cc5-81840b134811/486fed97-cc29-a85e-49e2-733c526b6b7f"
-					(reference "#PWR0140") (unit 1)
+					(reference "#PWR0144") (unit 1)
 				)
 			)
@@
 		(unit 1)
 		(exclude_from_sim no) (in_bom no) (on_board yes) (dnp no)
-		(property "Reference" "#PWR0141"
+		(property "Reference" "#PWR0145"
 			(at 60.96 39.37 0)
 			(effects (font (size 1.27 1.27)) (hide yes))
@@
 			(project "LFX_FC_R2"
 				(path "/9564b83f-500d-c692-1cc5-81840b134811/486fed97-cc29-a85e-49e2-733c526b6b7f"
-					(reference "#PWR0141") (unit 1)
+					(reference "#PWR0145") (unit 1)
 				)
 			)
@@
 		(unit 1)
 		(exclude_from_sim no) (in_bom no) (on_board yes) (dnp no)
-		(property "Reference" "#PWR0142"
+		(property "Reference" "#PWR0146"
 			(at 114.3 57.15 0)
 			(effects (font (size 1.27 1.27)) (hide yes))
@@
 			(project "LFX_FC_R2"
 				(path "/9564b83f-500d-c692-1cc5-81840b134811/486fed97-cc29-a85e-49e2-733c526b6b7f"
-					(reference "#PWR0142") (unit 1)
+					(reference "#PWR0146") (unit 1)
 				)
 			)
@@
 		(unit 1)
 		(exclude_from_sim no) (in_bom no) (on_board yes) (dnp no)
-		(property "Reference" "#PWR0143"
+		(property "Reference" "#PWR0147"
 			(at 19.05 106.68 0)
 			(effects (font (size 1.27 1.27)) (hide yes))
@@
 			(project "LFX_FC_R2"
 				(path "/9564b83f-500d-c692-1cc5-81840b134811/486fed97-cc29-a85e-49e2-733c526b6b7f"
-					(reference "#PWR0143") (unit 1)
+					(reference "#PWR0147") (unit 1)
 				)
 			)
@@
 		(unit 1)
 		(exclude_from_sim no) (in_bom no) (on_board yes) (dnp no)
-		(property "Reference" "#PWR0144"
+		(property "Reference" "#PWR0148"
 			(at 40.64 107.95 0)
 			(effects (font (size 1.27 1.27)) (hide yes))
@@
 			(project "LFX_FC_R2"
 				(path "/9564b83f-500d-c692-1cc5-81840b134811/486fed97-cc29-a85e-49e2-733c526b6b7f"
-					(reference "#PWR0144") (unit 1)
+					(reference "#PWR0148") (unit 1)
 				)
 			)
@@
 		(unit 1)
 		(exclude_from_sim no) (in_bom no) (on_board yes) (dnp no)
-		(property "Reference" "#PWR0145"
+		(property "Reference" "#PWR0149"
 			(at 60.96 106.68 0)
 			(effects (font (size 1.27 1.27)) (hide yes))
@@
 			(project "LFX_FC_R2"
 				(path "/9564b83f-500d-c692-1cc5-81840b134811/486fed97-cc29-a85e-49e2-733c526b6b7f"
-					(reference "#PWR0145") (unit 1)
+					(reference "#PWR0149") (unit 1)
 				)
 			)
@@
 			(effects (font (size 1.27 1.27)) (hide yes))
 		)
-		(property "Description" "ESD at the SIM holder, 0.5 pF (HDM asks <= 15 pF); the four channels are alike, assigned in the order the lines pass it"
+		(property "Description" "ESD at the SIM holder, 0.5 pF (HDM asks <= 15 pF); the four channels are alike, assigned so RST/CLK reach R37/R38 below without crossing (route_critical.hand_route_sim)"
 			(at 44.45 139.7 0)
 			(effects (font (size 1.27 1.27)) (hide yes))
@@
 		(unit 1)
 		(exclude_from_sim no) (in_bom no) (on_board yes) (dnp no)
-		(property "Reference" "#PWR0146"
+		(property "Reference" "#PWR0150"
 			(at 44.45 152.4 0)
 			(effects (font (size 1.27 1.27)) (hide yes))
@@
 			(project "LFX_FC_R2"
 				(path "/9564b83f-500d-c692-1cc5-81840b134811/486fed97-cc29-a85e-49e2-733c526b6b7f"
-					(reference "#PWR0146") (unit 1)
+					(reference "#PWR0150") (unit 1)
 				)
 			)
@@
 		(stroke (width 0) (type default))
 	)
+	(global_label "SIM_RST"
+		(shape bidirectional)
+		(at 60.96 137.16 0)
+		(effects (font (size 1.27 1.27)) (justify left))
+		(property "Intersheetrefs" "${INTERSHEET_REFS}"
+			(at 60.96 137.16 0)
+			(effects (font (size 1.27 1.27)) (hide yes))
+		)
+	)
+	(wire
+		(pts (xy 57.15 142.24) (xy 60.96 142.24))
+		(stroke (width 0) (type default))
+	)
 	(global_label "SIM_CLK"
-		(shape bidirectional)
-		(at 60.96 137.16 0)
-		(effects (font (size 1.27 1.27)) (justify left))
-		(property "Intersheetrefs" "${INTERSHEET_REFS}"
-			(at 60.96 137.16 0)
-			(effects (font (size 1.27 1.27)) (hide yes))
-		)
-	)
-	(wire
-		(pts (xy 57.15 142.24) (xy 60.96 142.24))
-		(stroke (width 0) (type default))
-	)
-	(global_label "SIM_RST"
 		(shape bidirectional)
 		(at 60.96 142.24 0)
@@
 		(unit 1)
 		(exclude_from_sim no) (in_bom no) (on_board yes) (dnp no)
-		(property "Reference" "#PWR0147"
+		(property "Reference" "#PWR0151"
 			(at 170.18 43.18 0)
 			(effects (font (size 1.27 1.27)) (hide yes))
@@
 			(project "LFX_FC_R2"
 				(path "/9564b83f-500d-c692-1cc5-81840b134811/486fed97-cc29-a85e-49e2-733c526b6b7f"
-					(reference "#PWR0147") (unit 1)
+					(reference "#PWR0151") (unit 1)
 				)
 			)
@@
 		(unit 1)
 		(exclude_from_sim no) (in_bom no) (on_board yes) (dnp no)
-		(property "Reference" "#PWR0148"
+		(property "Reference" "#PWR0152"
 			(at 181.61 57.15 0)
 			(effects (font (size 1.27 1.27)) (hide yes))
@@
 			(project "LFX_FC_R2"
 				(path "/9564b83f-500d-c692-1cc5-81840b134811/486fed97-cc29-a85e-49e2-733c526b6b7f"
-					(reference "#PWR0148") (unit 1)
+					(reference "#PWR0152") (unit 1)
 				)
 			)
@@
 		(unit 1)
 		(exclude_from_sim no) (in_bom no) (on_board yes) (dnp no)
-		(property "Reference" "#PWR0149"
+		(property "Reference" "#PWR0153"
 			(at 208.28 58.42 0)
 			(effects (font (size 1.27 1.27)) (hide yes))
@@
 			(project "LFX_FC_R2"
 				(path "/9564b83f-500d-c692-1cc5-81840b134811/486fed97-cc29-a85e-49e2-733c526b6b7f"
-					(reference "#PWR0149") (unit 1)
+					(reference "#PWR0153") (unit 1)
 				)
 			)
@@
 		(unit 1)
 		(exclude_from_sim no) (in_bom no) (on_board yes) (dnp no)
-		(property "Reference" "#PWR0150"
+		(property "Reference" "#PWR0154"
 			(at 303.53 43.18 0)
 			(effects (font (size 1.27 1.27)) (hide yes))
@@
 			(project "LFX_FC_R2"
 				(path "/9564b83f-500d-c692-1cc5-81840b134811/486fed97-cc29-a85e-49e2-733c526b6b7f"
-					(reference "#PWR0150") (unit 1)
+					(reference "#PWR0154") (unit 1)
 				)
 			)
@@
 		(unit 1)
 		(exclude_from_sim no) (in_bom no) (on_board yes) (dnp no)
-		(property "Reference" "#PWR0151"
+		(property "Reference" "#PWR0155"
 			(at 314.96 58.42 0)
 			(effects (font (size 1.27 1.27)) (hide yes))
@@
 			(project "LFX_FC_R2"
 				(path "/9564b83f-500d-c692-1cc5-81840b134811/486fed97-cc29-a85e-49e2-733c526b6b7f"
-					(reference "#PWR0151") (unit 1)
+					(reference "#PWR0155") (unit 1)
 				)
 			)
@@
 		(unit 1)
 		(exclude_from_sim no) (in_bom no) (on_board yes) (dnp no)
-		(property "Reference" "#PWR0152"
+		(property "Reference" "#PWR0156"
 			(at 341.63 59.69 0)
 			(effects (font (size 1.27 1.27)) (hide yes))
@@
 			(project "LFX_FC_R2"
 				(path "/9564b83f-500d-c692-1cc5-81840b134811/486fed97-cc29-a85e-49e2-733c526b6b7f"
-					(reference "#PWR0152") (unit 1)
+					(reference "#PWR0156") (unit 1)
 				)
 			)
@@
 		(unit 1)
 		(exclude_from_sim no) (in_bom no) (on_board yes) (dnp no)
-		(property "Reference" "#PWR0153"
+		(property "Reference" "#PWR0157"
 			(at 374.65 58.42 0)
 			(effects (font (size 1.27 1.27)) (hide yes))
@@
 			(project "LFX_FC_R2"
 				(path "/9564b83f-500d-c692-1cc5-81840b134811/486fed97-cc29-a85e-49e2-733c526b6b7f"
-					(reference "#PWR0153") (unit 1)
+					(reference "#PWR0157") (unit 1)
 				)
 			)
@@
 		(unit 1)
 		(exclude_from_sim no) (in_bom no) (on_board yes) (dnp no)
-		(property "Reference" "#PWR0154"
+		(property "Reference" "#PWR0158"
 			(at 284.48 109.22 0)
 			(effects (font (size 1.27 1.27)) (hide yes))
@@
 			(project "LFX_FC_R2"
 				(path "/9564b83f-500d-c692-1cc5-81840b134811/486fed97-cc29-a85e-49e2-733c526b6b7f"
-					(reference "#PWR0154") (unit 1)
-				)
-			)
+					(reference "#PWR0158") (unit 1)
+				)
+			)
